Commit message: Add differential drive robot description files and updated simple_robot description.

File: ros2_tutorial/src/robot_description/urdf/gem_robot.xacro (robot description, xacro)
@@ -1,3 +1,10 @@
+<?xml version="1.0"?>
 <robot name="simple_robot" xmlns:xacro="http://www.ros.org/wiki/xacro">
+  <material name="gray">
+    <color rgba="0.5 0.5 0.5 1.0"/>
+  </material>
+  <material name="black">
+    <color rgba="0.0 0.0 0.0 1.0"/>
+  </material>
   <xacro:property name="wheel_radius" value="0.1"/>
   <xacro:property name="wheel_width" value="0.05"/>
@@ -30,5 +37,5 @@
   </xacro:macro>
   <xacro:wheel name="left_wheel" y_offset="${wheel_offset_y}"/>
-  <xacro:wheel name="right_wheel" y_offset="-${wheel_offset_y}"/>
+  <xacro:wheel name="right_wheel" y_offset="${-wheel_offset_y}"/>
   <link name="lidar_link">
     <visual>
@@ -44,29 +51,3 @@
     <origin xyz="0.0 0.0 0.10" rpy="0.0 0.0 0.0"/>
   </joint>
-  <link name="camera_link">
-    <visual>
-      <geometry>
-        <box size="0.1 0.05 0.05"/>
-      </geometry>
-      <material name="black"/>
-    </visual>
-  </link>
-  <joint name="camera_joint" type="fixed">
-    <parent link="base_link"/>
-    <child link="camera_link"/>
-    <origin xyz="0.10 0.0 0.05" rpy="0.0 0.0 0.0"/>
-  </joint>
-  <link name="camera_optical_frame">
-    <visual>
-      <geometry>
-        <box size="0.05 0.05 0.05"/>
-      </geometry>
-      <material name="black"/>
-    </visual>
-  </link>
-  <joint name="camera_optical_frame_joint" type="fixed">
-    <parent link="camera_link"/>
-    <child link="camera_optical_frame"/>
-    <origin xyz="0.0 0.0 0.0" rpy="-1.5708 0.0 -1.5708"/>
-  </joint>
 </robot>

File: ros2_tutorial/src/robot_description/urdf/simple_robot.urdf (robot description, URDF)
Before this commit: robot simple_robot, 3 links, 2 joints
Links:
- removed link left_wheel_link
- removed link right_wheel_link
- added link camera_link; visual box size=0.1 0.05 0.05
- added link camera_optical_frame; visual box size=0.05 0.05 0.05
- added link left_wheel; visual cylinder length=0.05 radius=0.1
- added link lidar_link; visual cylinder length=0.1 radius=0.05
- added link right_wheel; visual cylinder length=0.05 radius=0.1
Joints:
- added joint camera_joint: type fixed, parent base_link, child camera_link, origin xyz=0.10 0.0 0.05 rpy=0.0 0.0 0.0
- added joint camera_optical_frame_joint: type fixed, parent camera_link, child camera_optical_frame, origin xyz=0.0 0.0 0.0 rpy=-1.5708 0.0 -1.5708
- added joint lidar_joint: type fixed, parent base_link, child lidar_link, origin xyz=0.0 0.0 0.10 rpy=0.0 0.0 0.0
- joint left_wheel_joint: child left_wheel_link -> left_wheel; origin xyz=0.0 0.225 0.1 rpy=0.0 0.0 0.0 -> xyz=0.0 0.225 -0.05 rpy=0.0 0.0 0.0
- joint right_wheel_joint: child right_wheel_link -> right_wheel; origin xyz=0.0 -0.225 0.1 rpy=0.0 0.0 0.0 -> xyz=0.0 -0.225 -0.05 rpy=0.0 0.0 0.0
